File: kicad/pressure_conditioner.kicad_sch (KiCad schematic)
At the start: 0 parts

Commit message: started top level file and channel components
Parts:
- added J1, J2, J3, J4, J5, J6, J7: 5023520201, CONN_SD-502352-001_02_MOL, symbol Pressure:5023520201
- added U1: (no value), CONN_SD-502352-001_02_MOL, symbol Pressure:NMK2415SAC
Connections:
- new net +15V: U1.5 (-V_out)
- new net +24V: J1.1, U1.1 (+V_in)
- new net -15V: U1.7 (+V_out)
- new net GND: J1.2, J2.2, J3.2, J4.2, J5.2, J6.2, J7.2, U1.2 (-V_in), U1.6 (0V_out)
