File: kicad/pressure_conditioner.kicad_pcb (KiCad board)
At the start: 2 copper layers, 0 parts

Commit message: began pcb layout
Parts:
- added C1: 1u, Capacitor_SMD:C_0805_2012Metric_Pad1.18x1.45mm_HandSolder, F.Cu at (155.0, 131.0)
- added C2: 1u, Capacitor_SMD:C_0805_2012Metric_Pad1.18x1.45mm_HandSolder, F.Cu at (158.0, 101.0)
- added C3: 1u, Capacitor_SMD:C_0805_2012Metric_Pad1.18x1.45mm_HandSolder, F.Cu at (154.9, 140.0)
- added C4: 1u, Capacitor_SMD:C_0805_2012Metric_Pad1.18x1.45mm_HandSolder, F.Cu at (155.0, 137.5)
- added C5: 1u, Capacitor_SMD:C_0805_2012Metric_Pad1.18x1.45mm_HandSolder, F.Cu at (155.0, 134.5)
- added C6: 1u, Capacitor_SMD:C_0805_2012Metric_Pad1.18x1.45mm_HandSolder, F.Cu at (154.9, 143.0)
- added D1: TVS, Diode_SMD:D_SMB, F.Cu at (50.0, 185.5)
- added D2: TVS, Diode_SMD:D_SMB, F.Cu at (72.5, 185.5)
- added D3: TVS, Diode_SMD:D_SMB, F.Cu at (94.9, 185.5)
- added J1: 24V Power Conn, Pressure:MOLEX_5023520201_2_Wire_DuraClik, F.Cu at (145.0, 67.0)
- added J2: P1 Vout Conn, Pressure:MOLEX_5023520201_2_Wire_DuraClik, F.Cu at (189.0, 70.0)
- added J3: P2 Vout Conn, Pressure:MOLEX_5023520201_2_Wire_DuraClik, F.Cu at (189.0, 88.0)
- added J4: P3 Vout Conn, Pressure:MOLEX_5023520201_2_Wire_DuraClik, F.Cu at (189.0, 106.0)
- added J5: P3 Sensor Conn, Pressure:MOLEX_5023520201_2_Wire_DuraClik, F.Cu at (125.0, 106.0)
- added J6: P2 Sensor Conn, Pressure:MOLEX_5023520201_2_Wire_DuraClik, F.Cu at (125.0, 88.0)
- added J7: P1 Sensor Conn, Pressure:MOLEX_5023520201_2_Wire_DuraClik, F.Cu at (125.0, 70.0)
- added R1: 47, Resistor_SMD:R_2512_6332Metric_Pad1.40x3.35mm_HandSolder, F.Cu at (39.4, 190.4)
- added R2: 47, Resistor_SMD:R_2512_6332Metric_Pad1.40x3.35mm_HandSolder, F.Cu at (61.8, 190.4)
- added R3: 47, Resistor_SMD:R_2512_6332Metric_Pad1.40x3.35mm_HandSolder, F.Cu at (84.3, 190.4)
- added U1: 24V +-15V Converter, Pressure:Murata_24-+-15_Conv_NMK2415SC, F.Cu at (161.0, 64.0)
- added U2: ~, Package_DIP:DIP-16_W7.62mm, F.Cu at (149.1, 84.8)
- added U3: ~, Package_DIP:DIP-16_W7.62mm, F.Cu at (149.3, 98.2)
- added U4: ~, Package_DIP:DIP-16_W7.62mm, F.Cu at (148.8, 111.6)
Other:
- board outline added: 85 x 56 mm

Commit message: Finished preliminary layout of Rev. A of board
Parts:
- removed U1: 24V +-15V Converter, Pressure:Murata_24-+-15_Conv_NMK2415SC
- added G***: LOGO, LOGO, F.Cu at (251.0, 37.8)
- added PS1: NMK2415SC, Pressure:Murata_24-+-15_Conv_NMK2415SC, F.Cu at (213.1, 42.3)
- U2, U3, U4: footprint Package_DIP:DIP-16_W7.62mm -> Package_DIP:CERDIP-16_W7.62mm_SideBrazed
- moved R1 148.9 mm to (124.1, 68.0)
- moved D1 130.6 mm to (124.2, 78.0)
- moved R2 119.9 mm to (124.1, 88.0)
- moved J2 106.9 mm to (295.0, 56.0)
- moved J4 106.6 mm to (295.0, 117.0)
- moved J3 106.1 mm to (295.0, 85.0)
- moved D2 101.6 mm to (124.2, 98.0)
- moved R3 91.5 mm to (124.1, 108.0)
- moved C1 73.7 mm to (142.2, 58.4)
- moved D3 73.6 mm to (124.2, 118.0)
- moved C4 66.3 mm to (150.2, 71.4)
- moved C3 43.8 mm to (142.4, 98.0)
- moved C5 42.6 mm to (150.4, 92.2)
- moved J1 33.5 mm to (155.0, 35.0)
- moved C6 31.4 mm to (150.4, 112.0)
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Connections:
- C4 pad 1: +15V -> -15V
- C5 pad 1: +15V -> -15V
- C6 pad 1: +15V -> -15V
- J4 pad 1: /Vout_P2 -> /Vout_P3
- U2 pad 4: +15V -> -15V
- U3 pad 4: +15V -> -15V
- U4 pad 4: +15V -> -15V
Routing:
- net GND: track 0.00 -> 472.1 mm, vias 0 -> 7
- net +15V: track 0.00 -> 221.9 mm
- net +24V: track 0.00 -> 205.0 mm
- net -15V: track 0.00 -> 178.0 mm
- net /Vout_P3: track 0.00 -> 156.6 mm
- net /Vout_P2: track 0.00 -> 151.9 mm
- net /Vout_P1: track 0.00 -> 150.6 mm
- net /I_P1: track 0.00 -> 33.7 mm
- net /I_P3: track 0.00 -> 25.3 mm
- net /I_P2: track 0.00 -> 23.8 mm
- net Net-(U2-+In): track 0.00 -> 22.9 mm
- net Net-(U4-+In): track 0.00 -> 22.4 mm
- net Net-(U3-+In): track 0.00 -> 22.3 mm
Other:
- board size 85 x 56 mm -> 200 x 200 mm
- board text added: "- +"
- board text added: "24V Conn"
- board text added: "P1 Sens Conn"
- board text added: "P1 Vout Conn"
- board text added: "P2 Sens Conn"
- board text added: "P2 Vout Conn"
- board text added: "P3 Sens Conn"
- board text added: "P3 Vout Conn"
- board text added: "Pressure Sensor Signal Conditioner 3 Channel 4-20mA Input 0-5V Output"
- board text added: "Rev. A"
