File: kicad/_restore_backup_2026-10-07T19-47-45-211/pressure_conditioner.kicad_sch (KiCad schematic)
At the start: 8 parts, among them J1 5023520201, J2 5023520201, J3 5023520201, J4 5023520201, J5 5023520201, J6 5023520201, J7 5023520201

Commit message: channel components, continued add from last commit
Other:
- removed sheet Pressure_Channel
Changed lines of the file:
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@@
-		)
-	)
-	(sheet
-		(at 83.82 66.04)
-		(size 48.26 33.02)
-		(exclude_from_sim no)
-		(in_bom yes)
-		(on_board yes)
-		(dnp no)
-		(fields_autoplaced yes)
-		(stroke
-			(width 0.1524)
-			(type solid)
-		)
-		(fill
-			(color 0 0 0 0)
-		)
-		(property "Sheetname" "Pressure_Channel"
-			(at 83.82 65.3284 0)
-			(show_name no)
-			(do_not_autoplace no)
-			(effects
-				(font
-					(size 1.27 1.27)
-				)
-				(justify left bottom)
-			)
-		)
-		(property "Sheetfile" "Pressure_Channel.kicad_sch"
-			(at 83.82 99.6446 0)
-			(show_name no)
-			(do_not_autoplace no)
-			(effects
-				(font
-					(size 1.27 1.27)
-				)
-				(justify left top)
-			)
-		)
-		(instances
-			(project "pressure_conditioner"
-				(path "/d1a2bab1-03ca-4de0-a936-00ed771cb4f3"
-					(page "2")
-				)
-			)
 		)
 	)
